Commit message: small changes

File: urdf_models/panda/panda_arm_box.urdf (robot description, URDF)
Before this commit: robot panda, 9 links, 8 joints
Links:
- link end-effector: geometry collision box size=0.25 0.20 0.02; visual box size=0.25 0.20 0.02
Joints:
- joint joint_ee: origin xyz=0 0 0.14 rpy=0 0 0 -> xyz=0.08 0 0.12 rpy=0 0 0

Commit message: moving up and down

File: urdf_models/panda/panda_arm_box.urdf (robot description, URDF)
Before this commit: robot panda, 9 links, 8 joints
Links:
- link end-effector: geometry collision box size=0.35 0.15 0.02; visual box size=0.35 0.15 0.02

Commit message: up down

File: urdf_models/panda/panda_arm_box.urdf (robot description, URDF)
Before this commit: robot panda, 9 links, 8 joints
Joints:
- joint joint_ee: origin xyz=0.08 0 0.12 rpy=0 0 0 -> xyz=0.1 0 0.12 rpy=0 0 0

Commit message: added plotting ball position to compare with ball position

File: urdf_models/panda/panda_arm_box.urdf (robot description, URDF)
Before this commit: robot panda, 9 links, 8 joints
Links:
- link end-effector: geometry collision box size=0.34 0.15 0.02; visual box size=0.34 0.15 0.02

Commit message: fixed to launch controller first, centered ball pos in ee

File: urdf_models/panda/panda_arm_box.urdf (robot description, URDF)
Before this commit: robot panda, 9 links, 8 joints
Links:
- link end-effector: geometry collision box size=0.38 0.15 0.02; visual box size=0.34 0.15 0.02
Joints:
- joint joint_ee: origin xyz=0.1 0 0.12 rpy=0 0 0 -> xyz=0.13 0 0.12 rpy=0 0 0

Commit message: testing on real robot and computer vision

File: urdf_models/panda/panda_arm_box.urdf (robot description, URDF)
Before this commit: robot panda, 9 links, 8 joints
Joints:
- joint joint_ee: origin xyz=0.13 0 0.12 rpy=0 0 0 -> xyz=0.13 0 0.12 rpy=0 0 -0.785

Commit message: more test

File: urdf_models/panda/panda_arm_box.urdf (robot description, URDF)
Before this commit: robot panda, 9 links, 8 joints
Joints:
- joint joint_ee: origin xyz=0.13 0 0.12 rpy=0 0 -0.785 -> xyz=0.1 -0.1 0.12 rpy=0 0 -0.785

Commit message: added mass matrix

File: urdf_models/panda/panda_arm_box.urdf (robot description, URDF)
Before this commit: robot panda, 9 links, 8 joints
Joints:
- joint joint_ee: origin xyz=0.1 -0.1 0.12 rpy=0 0 -0.785 -> xyz=0.0 0.0 0.0 rpy=0 0 0.785

Commit message: bounding box sim

File: urdf_models/panda/panda_arm_box.urdf (robot description, URDF)
Before this commit: robot panda, 9 links, 8 joints
Links:
- link end-effector: geometry collision box size=0.50 0.20 0.02; visual box size=0.50 0.20 0.02
Joints:
- joint joint_ee: origin xyz=0.0 0.0 0.0 rpy=0 0 0.785 -> xyz=0.0 0.0 0.12 rpy=0 0 0.785

Commit message: moved ee box shape 10 cm

File: urdf_models/panda/panda_arm_box.urdf (robot description, URDF)
Before this commit: robot panda, 9 links, 8 joints
Links:
- link end-effector: geometry collision box size=0.40 0.20 0.02; visual box size=0.40 0.20 0.02
